File: hardware/module-development-boards/type1/module_dev1.kicad_pcb (KiCad board)
At the start: 2 copper layers, 30 x 26 mm, 34 parts, among them J1 SensorHub_Module_CONN_V1, J10 Conn_01x04, J11 Conn_01x04, J12 Conn_01x01, J13 Conn_01x01, J14 Conn_01x01, J15 Conn_01x01, J16 Conn_01x01, J17 Conn_01x01, J18 Conn_01x01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

Commit message: cleanup dev board type 1
Parts:
- J1: value SensorHub_Module_CONN_V1 -> LegoSENSE_Module_CONN_V1
Other:
- board text added: "LegoSENSE Module Dev Board V1.0"
- board text removed: "SensorHub Module Dev Board V1.0 Scott Zhao 10/12/2021"
Changed lines of the file:
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@@
       (effects (font (size 0.6 0.6) (thickness 0.08)) (justify mirror))
     )
-    (fp_text value "SensorHub_Module_CONN_V1" (at 1.0035 -4) (layer "B.SilkS") hide
+    (fp_text value "LegoSENSE_Module_CONN_V1" (at 1.0035 -4) (layer "B.SilkS") hide
       (effects (font (size 0.6 0.6) (thickness 0.08)) (justify mirror))
     )
@@
   (gr_line (start 91.995 86.938) (end 121.995 86.938) (layer "Edge.Cuts") (width 0.05))
   (gr_line (start 121.995 86.938) (end 121.995 60.938) (layer "Edge.Cuts") (width 0.05))
-  (gr_text "SensorHub Module\nDev Board V1.0\nScott Zhao\n10/12/2021" (at 106.68 74.93 90) (layer "B.SilkS")
+  (gr_text "LegoSENSE Module\nDev Board V1.0" (at 106.68 74.93 90) (layer "B.SilkS")
     (effects (font (size 0.8 0.8) (thickness 0.15)) (justify left mirror))
   )
@@
     (priority 1)
     (connect_pads (clearance 0.508))
-    (min_thickness 0.254)
+    (min_thickness 0.254) (filled_areas_thickness no)
     (fill yes (thermal_gap 0.508) (thermal_bridge_width 0.508))
     (polygon
@@
     (priority 1)
     (connect_pads (clearance 0.508))
-    (min_thickness 0.254)
+    (min_thickness 0.254) (filled_areas_thickness no)
     (fill yes (thermal_gap 0.508) (thermal_bridge_width 0.508))
     (polygon
@@
   (zone (net 0) (net_name "") (layer "B.Mask") (hatch edge 0.508)
     (connect_pads (clearance 0.508))
-    (min_thickness 0.254)
+    (min_thickness 0.254) (filled_areas_thickness no)
     (fill yes (thermal_gap 0.508) (thermal_bridge_width 0.508))
     (polygon
@@
   (zone (net 0) (net_name "") (layer "B.Mask") (hatch edge 0.508)
     (connect_pads (clearance 0.508))
-    (min_thickness 0.254)
+    (min_thickness 0.254) (filled_areas_thickness no)
     (fill yes (thermal_gap 0.508) (thermal_bridge_width 0.508))
     (polygon
